Commit message: Version 2 du 15 avril 2022

File: urdf/actuators.xacro (robot description, xacro)
@@ -9,21 +9,41 @@
     -->
 <!-- Moteur F1 -->
+<!-- V2
 <xacro:thruster_macro namespace="${namespace}" thruster_id="0">
-    <origin xyz="-0.144 0.204 0.198" rpy="0 0 ${-45*d2r}" />
+    <origin xyz="0.128911 -0.168186 -0.198264" rpy="${90*d2r} 0 ${45*d2r}" />
 </xacro:thruster_macro>
 <xacro:thruster_macro namespace="${namespace}" thruster_id="1">
-    <origin xyz="0.164 0.204 -0.198" rpy="0 0 ${-135*d2r}" />
+    <origin xyz="-0.108871 -0.168186 -0.198264" rpy="${90*d2r} 0 ${-45*d2r}" />
 </xacro:thruster_macro>
 <xacro:thruster_macro namespace="${namespace}" thruster_id="2">
-    <origin xyz="0.164 -0.204 -0.198" rpy="0 0 ${135*d2r}" />
+    <origin xyz="-0.108871 0.168186 -0.198264" rpy="${-90*d2r} 0 ${45*d2r}" />
 </xacro:thruster_macro>
 <xacro:thruster_macro namespace="${namespace}" thruster_id="3">
-    <origin xyz="-0.144 -0.204 -0.198" rpy="0 0 ${45*d2r}" />
+    <origin xyz="0.128911 0.168186 -0.198264" rpy="${-90*d2r} 0 ${-45*d2r}" />
 </xacro:thruster_macro>
 <xacro:thruster_macro namespace="${namespace}" thruster_id="4">
-    <origin xyz="-0.083 0.144 0.184" rpy="${-90*d2r} 0 0" />
+    <origin xyz="-0.019275 -0.144590 0.133603" rpy="0 0 0" />
 </xacro:thruster_macro>
 <xacro:thruster_macro namespace="${namespace}" thruster_id="5">
-    <origin xyz="-0.019 -0.144 0.184" rpy="${-90*d2r} 0 0" />
+    <origin xyz="-0.083455 0.144590 0.133603" rpy="0 0 0" />
+</xacro:thruster_macro>
+-->
+<xacro:thruster_macro namespace="${namespace}" thruster_id="0">
+    <origin xyz="0.128911 -0.168186 -0.198264" rpy="${180*d2r} 0 ${-45*d2r}" />
+</xacro:thruster_macro>
+<xacro:thruster_macro namespace="${namespace}" thruster_id="1">
+    <origin xyz="-0.108871 -0.168186 -0.198264" rpy="${180*d2r} 0 ${45*d2r}" />
+</xacro:thruster_macro>
+<xacro:thruster_macro namespace="${namespace}" thruster_id="2">
+    <origin xyz="-0.108871 0.168186 -0.198264" rpy="0 0 ${-45*d2r}" />
+</xacro:thruster_macro>
+<xacro:thruster_macro namespace="${namespace}" thruster_id="3">
+    <origin xyz="0.128911 0.168186 -0.198264" rpy="0 0 ${45*d2r}" />
+</xacro:thruster_macro>
+<xacro:thruster_macro namespace="${namespace}" thruster_id="4">
+    <origin xyz="-0.019275 -0.144590 0.133603" rpy="0 0 0" />
+</xacro:thruster_macro>
+<xacro:thruster_macro namespace="${namespace}" thruster_id="5">
+    <origin xyz="-0.083455 0.144590 0.133603" rpy="0 0 0" />
 </xacro:thruster_macro>
 </robot>

File: urdf/base.xacro (robot description, xacro)
@@ -25,5 +25,5 @@
     Open the meshes for the RexROV vehicle in Blender to see an example on the mesh placement.
   -->
-  <xacro:property name="visual_mesh_file" value="file://$(find divy2_description)/meshes/divy_base_no_propeller.dae"/>
+  <xacro:property name="visual_mesh_file" value="file://$(find divy2_description)/meshes/divy_base_no_propeller_modif3.dae"/>
   <!-- Collision geometry mesh, usually in STL format (it is recommended to keep
   this geometry as simple as possible to improve the performance the physics engine

File: urdf/gazebo.xacro (robot description, xacro)
@@ -6,7 +6,7 @@
     <xacro:property name="divy2_volume" value="0.0199420"/>
     <!-- Describing the dimensions of the vehicle's bounding box -->
-    <xacro:property name="divy2_length" value="0.425"/>
-    <xacro:property name="divy2_width"  value="0.410"/>
-    <xacro:property name="divy2_height" value="0.480"/>
+    <xacro:property name="divy2_length" value="0.47307"/>
+    <xacro:property name="divy2_width"  value="0.43675"/>
+    <xacro:property name="divy2_height" value="0.42738"/>
     <xacro:macro name="divy2_hydro_model" params="namespace">
       <!-- List of hydrodynamic models this robot's links -->
@@ -37,10 +37,10 @@
           <type>fossen</type>
           <added_mass>
-            0 0 0 0 0 0
-            0 0 0 0 0 0
-            0 0 0 0 0 0
-            0 0 0 0 0 0
-            0 0 0 0 0 0
-            0 0 0 0 0 0
+            779.79 -6.8773 -103.32  8.5426 -165.54 -7.8033
+           -6.8773    1222   51.29  409.44 -5.8488  62.726
+           -103.32   51.29  3659.9  6.1112 -386.42  10.774
+            8.5426  409.44  6.1112   534.9 -10.027  21.019
+           -165.54 -5.8488 -386.42 -10.027  842.69 -1.1162
+           -7.8033  62.726  10.775  21.019 -1.1162  224.32
           </added_mass>
           <!--
@@ -49,5 +49,5 @@
           -->
           <linear_damping>
-            0 0 0 0 0 0
+              -74.82 -69.48 -728.4 -268.8 -309.77 -105
           </linear_damping>
           <!--
@@ -65,5 +65,5 @@
           -->
           <quadratic_damping>
-            0 0 0 0 0 0
+              -748.22 -992.53 -1821.01 -672 -774.44 -523.27
           </quadratic_damping>
           <!--

Commit message: Version numéro 2 du robot, déplacements non fonctionnels mais code d'envoie aux moteurs fonctionnels

File: urdf/actuators.xacro (robot description, xacro)
@@ -42,8 +42,8 @@
 </xacro:thruster_macro>
 <xacro:thruster_macro namespace="${namespace}" thruster_id="4">
-    <origin xyz="-0.019275 -0.144590 0.133603" rpy="0 0 0" />
+    <origin xyz="-0.019275 -0.144590 0.133603" rpy="0 ${90*d2r} 0" />
 </xacro:thruster_macro>
 <xacro:thruster_macro namespace="${namespace}" thruster_id="5">
-    <origin xyz="-0.083455 0.144590 0.133603" rpy="0 0 0" />
+    <origin xyz="-0.083455 0.144590 0.133603" rpy="0 ${90*d2r} 0" />
 </xacro:thruster_macro>
 </robot>

File: urdf/base.xacro (robot description, xacro)
@@ -25,5 +25,5 @@
     Open the meshes for the RexROV vehicle in Blender to see an example on the mesh placement.
   -->
-  <xacro:property name="visual_mesh_file" value="file://$(find divy2_description)/meshes/divy_base_no_propeller_modif3.dae"/>
+  <xacro:property name="visual_mesh_file" value="file://$(find divy2_description)/meshes/Fdivy.dae"/>
   <!-- Collision geometry mesh, usually in STL format (it is recommended to keep
   this geometry as simple as possible to improve the performance the physics engine

Commit message: Modification des données physiques du robot, séance du 18/05/2022, problème sur le modèle inverse

File: urdf/actuators.xacro (robot description, xacro)
@@ -30,5 +30,5 @@
 -->
 <xacro:thruster_macro namespace="${namespace}" thruster_id="0">
-    <origin xyz="0.128911 -0.168186 -0.198264" rpy="${180*d2r} 0 ${-45*d2r}" />
+    <origin xyz="0.128911 -0.168186 -0.198264" rpy="${180*d2r} 0 ${135*d2r}" />
 </xacro:thruster_macro>
 <xacro:thruster_macro namespace="${namespace}" thruster_id="1">
@@ -39,11 +39,11 @@
 </xacro:thruster_macro>
 <xacro:thruster_macro namespace="${namespace}" thruster_id="3">
-    <origin xyz="0.128911 0.168186 -0.198264" rpy="0 0 ${45*d2r}" />
+    <origin xyz="0.128911 0.168186 -0.198264" rpy="0 0 ${-135*d2r}" />
 </xacro:thruster_macro>
 <xacro:thruster_macro namespace="${namespace}" thruster_id="4">
-    <origin xyz="-0.019275 -0.144590 0.133603" rpy="0 ${90*d2r} 0" />
+    <origin xyz="-0.019275 -0.144590 0.133603" rpy="0 ${-90*d2r} 0" />
 </xacro:thruster_macro>
 <xacro:thruster_macro namespace="${namespace}" thruster_id="5">
-    <origin xyz="-0.083455 0.144590 0.133603" rpy="0 ${90*d2r} 0" />
+    <origin xyz="-0.083455 0.144590 0.133603" rpy="0 ${-90*d2r} 0" />
 </xacro:thruster_macro>
 </robot>

File: urdf/base.xacro (robot description, xacro)
@@ -14,5 +14,6 @@
     Vehicle's parameters (remember to enter the model parameters below)
   -->
-  <xacro:property name="mass" value="10.3481054124272"/>
+  <xacro:property name="mass" value="12.647150"/>
+  <!--<xacro:property name="mass" value="10.3481054124272"/> -->
   <!-- Center of gravity -->
   <!-- <xacro:property name="cog" value="0 0 0"/> -->
@@ -25,5 +26,5 @@
     Open the meshes for the RexROV vehicle in Blender to see an example on the mesh placement.
   -->
-  <xacro:property name="visual_mesh_file" value="file://$(find divy2_description)/meshes/Fdivy.dae"/>
+  <xacro:property name="visual_mesh_file" value="file://$(find divy2_description)/meshes/Fdivy_color.dae"/>
   <!-- Collision geometry mesh, usually in STL format (it is recommended to keep
   this geometry as simple as possible to improve the performance the physics engine
@@ -49,10 +50,10 @@
         -->
           <inertia
-          ixx="0.0492677110434437"
-          ixy="-0.00016910155817298"
-          ixz="-6.99314826205029E-05"
-          iyy="0.0507820794986514"
-          iyz="-3.82177497348897E-06"
-          izz="0.0455384747944849" />
+          ixx="0.350294"
+          ixy="-0.003760"
+          ixz="-0.011935"
+          iyy="0.422754"
+          iyz="-0.000109"
+          izz="0.324846" />
         </inertial>
         <!-- This visual geometry representation can be used when running
@@ -67,5 +68,5 @@
           <origin xyz="0 0 0" rpy="0 0 0"/>
           <geometry>
-            <box size="2.56 1.50 0.40"/>
+            <box size="1 1 1"/>
           </geometry>
         </collision>

File: urdf/gazebo.xacro (robot description, xacro)
@@ -2,7 +2,7 @@
 <robot xmlns:xacro="http://www.ros.org/wiki/xacro">
     <!-- Center of buoyancy -->
-    <xacro:property name="divy2_cob" value="-0.004150 -0.000219 -0.036355"/>
+    <xacro:property name="divy2_cob" value="-0.004148 0.000012 -0.036619"/>
     <!-- Vehicle's actual volume (Gazebo cannot compute the volume out of the mesh) -->
-    <xacro:property name="divy2_volume" value="0.0199420"/>
+    <xacro:property name="divy2_volume" value="0.019942"/>
     <!-- Describing the dimensions of the vehicle's bounding box -->
     <xacro:property name="divy2_length" value="0.47307"/>
@@ -44,4 +44,16 @@
            -7.8033  62.726  10.775  21.019 -1.1162  224.32
           </added_mass>
+          <!--
+          <hydrodynamic_model>
+            <type>fossen</type>
+            <added_mass>
+              1.7182 0 0 0 0 0
+              0 0 0 0 0 0
+              0 0 5.468 0 0 0
+              0 0 0 0 0 0
+              0 0 0 0 1.2481 0
+              0 0 0 0 0 0.4006
+            </added_mass>
+            -->
           <!--
             The linear damping coefficients can be provided as a diagonal (6 elements)

File: urdf/snippets.xacro (robot description, xacro)
@@ -25,5 +25,5 @@
         mesh_filename="file://$(find divy2_description)/meshes/propeller.dae"
       dyn_time_constant="0.05"
-      rotor_constant="0.026546960744430276">
+      rotor_constant="0.1">
       <xacro:insert_block name="origin"/>
     </xacro:thruster_module_first_order_basic_fcn_macro>
